Commit message: joint_state_publisher

File: src/auv_manipulator/urdf/manipulator.urdf.xacro (robot description, xacro)
@@ -1,12 +1,5 @@
 <?xml version="1.0"?>
-<robot name="auv_manipulator"
-  xmlns:xacro="http://ros.org/wiki/xacro">
-  <xacro:property name="width" value="0.2" />
-  <xacro:property name="leglen" value="0.6" />
-  <xacro:property name="polelen" value="0.2" />
-  <xacro:property name="bodylen" value="0.6" />
-  <xacro:property name="baselen" value="0.4" />
-  <xacro:property name="wheeldiam" value="0.07" />
-  <material name="blue">
+<robot name="visual">
+<material name="blue">
     <color rgba="0 0 0.8 1"/>
   </material>
@@ -17,173 +10,201 @@
     <color rgba="1 1 1 1"/>
   </material>
-  <xacro:macro name="default_inertial" params="mass">
-    <inertial>
-      <mass value="${mass}" />
-      <inertia ixx="1.0" ixy="0.0" ixz="0.0" iyy="1.0" iyz="0.0" izz="1.0" />
-    </inertial>
-  </xacro:macro>
   <link name="base_link">
     <visual>
       <geometry>
-        <cylinder radius="${width}" length="${bodylen}"/>
+        <cylinder length="0.6" radius="0.2"/>
       </geometry>
       <material name="blue"/>
     </visual>
-    <collision>
-      <geometry>
-        <cylinder radius="${width}" length="${bodylen}"/>
-      </geometry>
-    </collision>
-    <xacro:default_inertial mass="10"/>
-  </link>
-  <xacro:macro name="wheel" params="prefix suffix reflect">
-    <link name="${prefix}_${suffix}_wheel">
-      <visual>
-        <origin xyz="0 0 0" rpy="${pi/2} 0 0" />
-        <geometry>
-          <cylinder radius="${wheeldiam/2}" length="0.1"/>
-        </geometry>
-        <material name="black"/>
-      </visual>
-      <collision>
-        <origin xyz="0 0 0" rpy="${pi/2} 0 0" />
-        <geometry>
-          <cylinder radius="${wheeldiam/2}" length="0.1"/>
-        </geometry>
-      </collision>
-      <xacro:default_inertial mass="1"/>
-    </link>
-    <joint name="${prefix}_${suffix}_wheel_joint" type="continuous">
-      <axis xyz="0 1 0" rpy="0 0 0" />
-      <parent link="${prefix}_base"/>
-      <child link="${prefix}_${suffix}_wheel"/>
-      <origin xyz="${baselen*reflect/3} 0 -${wheeldiam/2+.05}" rpy="0 0 0"/>
-    </joint>
-  </xacro:macro>
-  <xacro:macro name="leg" params="prefix reflect">
-    <link name="${prefix}_leg">
-      <visual>
-        <geometry>
-          <box size="${leglen} 0.1 0.2"/>
-        </geometry>
-        <origin xyz="0 0 -${leglen/2}" rpy="0 ${pi/2} 0"/>
-        <material name="white"/>
-      </visual>
-      <collision>
-        <geometry>
-          <box size="${leglen} 0.1 0.2"/>
-        </geometry>
-        <origin xyz="0 0 -${leglen/2}" rpy="0 ${pi/2} 0"/>
-      </collision>
-      <xacro:default_inertial mass="10"/>
-    </link>
-    <joint name="base_to_${prefix}_leg" type="fixed">
-      <parent link="base_link"/>
-      <child link="${prefix}_leg"/>
-      <origin xyz="0 ${reflect*(width+.02)} 0.25" />
-    </joint>
-    <link name="${prefix}_base">
-      <visual>
-        <geometry>
-          <box size="${baselen} 0.1 0.1"/>
-        </geometry>
-        <material name="white"/>
-      </visual>
-      <collision>
-        <geometry>
-          <box size="${baselen} 0.1 0.1"/>
-        </geometry>
-      </collision>
-      <xacro:default_inertial mass="10"/>
-    </link>
-    <joint name="${prefix}_base_joint" type="fixed">
-      <parent link="${prefix}_leg"/>
-      <child link="${prefix}_base"/>
-      <origin xyz="0 0 ${-leglen}" />
-    </joint>
-    <xacro:wheel prefix="${prefix}" suffix="front" reflect="1"/>
-    <xacro:wheel prefix="${prefix}" suffix="back" reflect="-1"/>
-  </xacro:macro>
-  <xacro:leg prefix="right" reflect="-1" />
-  <xacro:leg prefix="left" reflect="1" />
+  </link>
+  <link name="right_leg">
+    <visual>
+      <geometry>
+        <box size="0.6 0.1 0.2"/>
+      </geometry>
+      <origin rpy="0 1.57075 0" xyz="0 0 -0.3"/>
+      <material name="white"/>
+    </visual>
+  </link>
+  <joint name="base_to_right_leg" type="fixed">
+    <parent link="base_link"/>
+    <child link="right_leg"/>
+    <origin xyz="0 -0.22 0.25"/>
+  </joint>
+  <link name="right_base">
+    <visual>
+      <geometry>
+        <box size="0.4 0.1 0.1"/>
+      </geometry>
+      <material name="white"/>
+    </visual>
+  </link>
+  <joint name="right_base_joint" type="fixed">
+    <parent link="right_leg"/>
+    <child link="right_base"/>
+    <origin xyz="0 0 -0.6"/>
+  </joint>
+  <link name="right_front_wheel">
+    <visual>
+      <origin rpy="1.57075 0 0" xyz="0 0 0"/>
+      <geometry>
+        <cylinder length="0.1" radius="0.035"/>
+      </geometry>
+      <material name="black"/>
+    </visual>
+  </link>
+  <joint name="right_front_wheel_joint" type="continuous">
+    <axis rpy="0 0 0" xyz="0 1 0"/>
+    <parent link="right_base"/>
+    <child link="right_front_wheel"/>
+    <origin rpy="0 0 0" xyz="0.133333333333 0 -0.085"/>
+  </joint>
+  <link name="right_back_wheel">
+    <visual>
+      <origin rpy="1.57075 0 0" xyz="0 0 0"/>
+      <geometry>
+        <cylinder length="0.1" radius="0.035"/>
+      </geometry>
+      <material name="black"/>
+    </visual>
+  </link>
+  <joint name="right_back_wheel_joint" type="continuous">
+    <axis rpy="0 0 0" xyz="0 1 0"/>
+    <parent link="right_base"/>
+    <child link="right_back_wheel"/>
+    <origin rpy="0 0 0" xyz="-0.133333333333 0 -0.085"/>
+  </joint>
+  <link name="left_leg">
+    <visual>
+      <geometry>
+        <box size="0.6 0.1 0.2"/>
+      </geometry>
+      <origin rpy="0 1.57075 0" xyz="0 0 -0.3"/>
+      <material name="white"/>
+    </visual>
+  </link>
+  <joint name="base_to_left_leg" type="fixed">
+    <parent link="base_link"/>
+    <child link="left_leg"/>
+    <origin xyz="0 0.22 0.25"/>
+  </joint>
+  <link name="left_base">
+    <visual>
+      <geometry>
+        <box size="0.4 0.1 0.1"/>
+      </geometry>
+      <material name="white"/>
+    </visual>
+  </link>
+  <joint name="left_base_joint" type="fixed">
+    <parent link="left_leg"/>
+    <child link="left_base"/>
+    <origin xyz="0 0 -0.6"/>
+  </joint>
+  <link name="left_front_wheel">
+    <visual>
+      <origin rpy="1.57075 0 0" xyz="0 0 0"/>
+      <geometry>
+        <cylinder length="0.1" radius="0.035"/>
+      </geometry>
+      <material name="black"/>
+    </visual>
+  </link>
+  <joint name="left_front_wheel_joint" type="continuous">
+    <axis rpy="0 0 0" xyz="0 1 0"/>
+    <parent link="left_base"/>
+    <child link="left_front_wheel"/>
+    <origin rpy="0 0 0" xyz="0.133333333333 0 -0.085"/>
+  </joint>
+  <link name="left_back_wheel">
+    <visual>
+      <origin rpy="1.57075 0 0" xyz="0 0 0"/>
+      <geometry>
+        <cylinder length="0.1" radius="0.035"/>
+      </geometry>
+      <material name="black"/>
+    </visual>
+  </link>
+  <joint name="left_back_wheel_joint" type="continuous">
+    <axis rpy="0 0 0" xyz="0 1 0"/>
+    <parent link="left_base"/>
+    <child link="left_back_wheel"/>
+    <origin rpy="0 0 0" xyz="-0.133333333333 0 -0.085"/>
+  </joint>
   <joint name="gripper_extension" type="prismatic">
     <parent link="base_link"/>
     <child link="gripper_pole"/>
-    <limit effort="1000.0" lower="-${width*2-.02}" upper="0" velocity="0.5"/>
-    <origin rpy="0 0 0" xyz="${width-.01} 0 0.2"/>
+    <limit effort="1000.0" lower="-0.38" upper="0" velocity="0.5"/>
+    <origin rpy="0 0 0" xyz="0.19 0 0.2"/>
   </joint>
   <link name="gripper_pole">
     <visual>
       <geometry>
-        <cylinder length="${polelen}" radius="0.01"/>
-      </geometry>
-      <origin xyz="${polelen/2} 0 0" rpy="0 ${pi/2} 0 "/>
-    </visual>
-    <collision>
-      <geometry>
-        <cylinder length="${polelen}" radius="0.01"/>
-      </geometry>
-      <origin xyz="${polelen/2} 0 0" rpy="0 ${pi/2} 0 "/>
-    </collision>
-    <xacro:default_inertial mass="0.05"/>
-  </link>
-  <xacro:macro name="gripper" params="prefix reflect">
-    <joint name="${prefix}_gripper_joint" type="revolute">
-      <axis xyz="0 0 ${reflect}"/>
-      <limit effort="1000.0" lower="0.0" upper="0.548" velocity="0.5"/>
-      <origin rpy="0 0 0" xyz="${polelen} ${reflect*0.01} 0"/>
-      <parent link="gripper_pole"/>
-      <child link="${prefix}_gripper"/>
-    </joint>
-    <link name="${prefix}_gripper">
-      <visual>
-        <origin rpy="${(reflect-1)/2*pi} 0 0" xyz="0 0 0"/>
-        <geometry>
-          <box size="0.05 0.01 0.01"/>
-        </geometry>
-      </visual>
-      <collision>
-        <geometry>
-          <box size="0.05 0.01 0.01"/>
-        </geometry>
-        <origin rpy="${(reflect-1)/2*pi} 0 0" xyz="0 0 0"/>
-      </collision>
-      <xacro:default_inertial mass="0.05"/>
-    </link>
-    <joint name="${prefix}_tip_joint" type="fixed">
-      <parent link="${prefix}_gripper"/>
-      <child link="${prefix}_tip"/>
-    </joint>
-    <link name="${prefix}_tip">
-      <visual>
-        <origin rpy="${(reflect-1)/2*pi} 0 0" xyz="0.09137 0.00495 0"/>
-        <geometry>
-          <box size="0.01 0.01 0.01"/>
-        </geometry>
-      </visual>
-      <collision>
-        <geometry>
-          <box size="0.01 0.01 0.01"/>
-        </geometry>
-        <origin rpy="${(reflect-1)/2*pi} 0 0" xyz="0.09137 0.00495 0"/>
-      </collision>
-      <xacro:default_inertial mass="0.05"/>
-    </link>
-  </xacro:macro>
-  <xacro:gripper prefix="left" reflect="1" />
-  <xacro:gripper prefix="right" reflect="-1" />
+        <cylinder length="0.2" radius="0.01"/>
+      </geometry>
+      <origin rpy="0 1.57075 0 " xyz="0.1 0 0"/>
+    </visual>
+  </link>
+  <joint name="left_gripper_joint" type="revolute">
+    <axis xyz="0 0 1"/>
+    <limit effort="1000.0" lower="0.0" upper="0.548" velocity="0.5"/>
+    <origin rpy="0 0 0" xyz="0.2 0.01 0"/>
+    <parent link="gripper_pole"/>
+    <child link="left_gripper"/>
+  </joint>
+  <link name="left_gripper">
+    <visual>
+      <origin rpy="0.0 0 0" xyz="0 0 0"/>
+      <geometry>
+        <mesh filename="package://urdf_tutorial/meshes/l_finger.dae"/>
+      </geometry>
+    </visual>
+  </link>
+  <joint name="left_tip_joint" type="fixed">
+    <parent link="left_gripper"/>
+    <child link="left_tip"/>
+  </joint>
+  <link name="left_tip">
+    <visual>
+      <origin rpy="0.0 0 0" xyz="0.09137 0.00495 0"/>
+      <geometry>
+        <mesh filename="package://urdf_tutorial/meshes/l_finger_tip.dae"/>
+      </geometry>
+    </visual>
+  </link>
+  <joint name="right_gripper_joint" type="revolute">
+    <axis xyz="0 0 -1"/>
+    <limit effort="1000.0" lower="0.0" upper="0.548" velocity="0.5"/>
+    <origin rpy="0 0 0" xyz="0.2 -0.01 0"/>
+    <parent link="gripper_pole"/>
+    <child link="right_gripper"/>
+  </joint>
+  <link name="right_gripper">
+    <visual>
+      <origin rpy="-3.1415 0 0" xyz="0 0 0"/>
+      <geometry>
+        <mesh filename="package://urdf_tutorial/meshes/l_finger.dae"/>
+      </geometry>
+    </visual>
+  </link>
+  <joint name="right_tip_joint" type="fixed">
+    <parent link="right_gripper"/>
+    <child link="right_tip"/>
+  </joint>
+  <link name="right_tip">
+    <visual>
+      <origin rpy="-3.1415 0 0" xyz="0.09137 0.00495 0"/>
+      <geometry>
+        <mesh filename="package://urdf_tutorial/meshes/l_finger_tip.dae"/>
+      </geometry>
+    </visual>
+  </link>
   <link name="head">
     <visual>
       <geometry>
-        <sphere radius="${width}"/>
-      </geometry>
-      <material name="white"/>
-    </visual>
-    <collision>
-      <geometry>
-        <sphere radius="${width}"/>
-      </geometry>
-    </collision>
-    <xacro:default_inertial mass="2"/>
+        <sphere radius="0.2"/>
+      </geometry>
+      <material name="white"/>
+    </visual>
   </link>
   <joint name="head_swivel" type="continuous">
@@ -191,5 +212,5 @@
     <child link="head"/>
     <axis xyz="0 0 1"/>
-    <origin xyz="0 0 ${bodylen/2}"/>
+    <origin xyz="0 0 0.3"/>
   </joint>
   <link name="box">
@@ -199,17 +220,10 @@
       </geometry>
       <material name="blue"/>
-      <origin xyz="-0.04 0 0"/>
-    </visual>
-    <collision>
-      <geometry>
-        <box size="0.08 0.08 0.08"/>
-      </geometry>
-    </collision>
-    <xacro:default_inertial mass="1"/>
+    </visual>
   </link>
   <joint name="tobox" type="fixed">
     <parent link="head"/>
     <child link="box"/>
-    <origin xyz="${.707*width+0.04} 0 ${.707*width}"/>
+    <origin xyz="0.1814 0 0.1414"/>
   </joint>
 </robot>
