Commit message: Adds urdf for manipulator

File: src/auv_manipulator/urdf/manipulator.urdf.xacro (robot description, xacro)
@@ -1,229 +1,160 @@
 <?xml version="1.0"?>
-<robot name="visual">
-<material name="blue">
-    <color rgba="0 0 0.8 1"/>
+<robot xmlns:xacro="http://www.ros.org/wiki/xacro" name="twig">
+  <xacro:property name="name" value="twig" />
+  <xacro:property name="base_length" value="0.08" />
+  <xacro:property name="base_radius" value="0.12" />
+  <xacro:property name="base_width" value="0.1" />
+  <xacro:property name="shoulder_length" value="0.2" />
+  <xacro:property name="shoulder_radius" value="0.05" />
+  <xacro:property name="wrist_length" value="0.01" />
+  <xacro:property name="wrist_radius" value="0.05" />
+  <xacro:property name="gripper_length" value="0.05" />
+  <xacro:property name="gripper_width" value="0.05" />
+  <xacro:property name="gripper_height" value="0.1" />
+  <xacro:property name="shoulder_limit" value="${(pi/180)*100}" />
+  <xacro:property name="wrist_limit" value="${(pi/180)*360}" />
+  <xacro:property name="gripper_limit" value="0.04" />
+  <material name="blue">
+    <color rgba="0 0 1 1" />
+  </material>
+  <material name="red">
+    <color rgba="1 0 0 1" />
   </material>
   <material name="black">
-    <color rgba="0 0 0 1"/>
+    <color rgba="0 0 0 1" />
   </material>
   <material name="white">
-    <color rgba="1 1 1 1"/>
+    <color rgba="1 1 1 1" />
+  </material>
+  <material name="grey">
+    <color rgba="0.5 0.5 0.5 1" />
   </material>
   <link name="base_link">
     <visual>
       <geometry>
-        <cylinder length="0.6" radius="0.2"/>
+        <cylinder length="1" radius="0.15" />
       </geometry>
-      <material name="blue"/>
+      <material name="grey" />
+      <origin rpy="0 ${pi/2} 0" />
     </visual>
+    <collision>
+      <geometry>
+        <cylinder length="1" radius="0.15" />
+      </geometry>
+      <origin rpy="0 ${pi/2} 0" />
+    </collision>
   </link>
-  <link name="right_leg">
+  <link name="${name}_base">
     <visual>
       <geometry>
-        <box size="0.6 0.1 0.2"/>
+        <cylinder length="${base_width}" radius="${base_radius}" />
       </geometry>
-      <origin rpy="0 1.57075 0" xyz="0 0 -0.3"/>
-      <material name="white"/>
+      <material name="grey" />
+      <origin rpy="0 ${pi/2} ${pi/2}" />
     </visual>
+    <collision>
+      <geometry>
+        <cylinder length="${base_width}" radius="${base_radius}" />
+      </geometry>
+      <origin rpy="0 ${pi/2} ${pi/2}" />
+    </collision>
   </link>
-  <joint name="base_to_right_leg" type="fixed">
-    <parent link="base_link"/>
-    <child link="right_leg"/>
-    <origin xyz="0 -0.22 0.25"/>
-  </joint>
-  <link name="right_base">
+  <link name="${name}_shoulder">
     <visual>
       <geometry>
-        <box size="0.4 0.1 0.1"/>
+        <cylinder length="${shoulder_length}" radius="${shoulder_radius}" />
       </geometry>
-      <material name="white"/>
+      <origin xyz="0 0 ${shoulder_length/2}" />
+      <material name="red" />
     </visual>
+    <collision>
+      <geometry>
+        <cylinder length="${shoulder_length}" radius="${shoulder_radius}" />
+      </geometry>
+      <origin xyz="0 0 ${shoulder_length/2}" />
+    </collision>
   </link>
-  <joint name="right_base_joint" type="fixed">
-    <parent link="right_leg"/>
-    <child link="right_base"/>
-    <origin xyz="0 0 -0.6"/>
-  </joint>
-  <link name="right_front_wheel">
-    <visual>
-      <origin rpy="1.57075 0 0" xyz="0 0 0"/>
-      <geometry>
-        <cylinder length="0.1" radius="0.035"/>
-      </geometry>
-      <material name="black"/>
-    </visual>
-  </link>
-  <joint name="right_front_wheel_joint" type="continuous">
-    <axis rpy="0 0 0" xyz="0 1 0"/>
-    <parent link="right_base"/>
-    <child link="right_front_wheel"/>
-    <origin rpy="0 0 0" xyz="0.133333333333 0 -0.085"/>
-  </joint>
-  <link name="right_back_wheel">
-    <visual>
-      <origin rpy="1.57075 0 0" xyz="0 0 0"/>
-      <geometry>
-        <cylinder length="0.1" radius="0.035"/>
-      </geometry>
-      <material name="black"/>
-    </visual>
-  </link>
-  <joint name="right_back_wheel_joint" type="continuous">
-    <axis rpy="0 0 0" xyz="0 1 0"/>
-    <parent link="right_base"/>
-    <child link="right_back_wheel"/>
-    <origin rpy="0 0 0" xyz="-0.133333333333 0 -0.085"/>
-  </joint>
-  <link name="left_leg">
+  <link name="${name}_wrist">
     <visual>
       <geometry>
-        <box size="0.6 0.1 0.2"/>
+        <cylinder length="${wrist_length}" radius="${wrist_radius}" />
       </geometry>
-      <origin rpy="0 1.57075 0" xyz="0 0 -0.3"/>
-      <material name="white"/>
+      <origin xyz="0 0 ${wrist_length/2}" />
+      <material name="white" />
     </visual>
+    <collision>
+      <geometry>
+        <cylinder length="${wrist_length}" radius="${wrist_radius}" />
+      </geometry>
+      <origin xyz="0 0 ${wrist_length/2}" />
+    </collision>
   </link>
-  <joint name="base_to_left_leg" type="fixed">
-    <parent link="base_link"/>
-    <child link="left_leg"/>
-    <origin xyz="0 0.22 0.25"/>
-  </joint>
-  <link name="left_base">
+  <link name="${name}_gripper">
+  </link>
+  <link name="${name}_left_gripper">
     <visual>
       <geometry>
-        <box size="0.4 0.1 0.1"/>
+        <box size="${gripper_length} ${gripper_width} ${gripper_height}" />
       </geometry>
-      <material name="white"/>
+      <origin xyz="${-gripper_length/2} 0 ${gripper_height/2}" />
+      <material name="blue" />
     </visual>
+    <collision>
+      <geometry>
+        <box size="${gripper_length} ${gripper_width} ${gripper_height}" />
+      </geometry>
+      <origin xyz="${-gripper_length/2} 0 ${gripper_height/2}" />
+    </collision>
   </link>
-  <joint name="left_base_joint" type="fixed">
-    <parent link="left_leg"/>
-    <child link="left_base"/>
-    <origin xyz="0 0 -0.6"/>
-  </joint>
-  <link name="left_front_wheel">
-    <visual>
-      <origin rpy="1.57075 0 0" xyz="0 0 0"/>
-      <geometry>
-        <cylinder length="0.1" radius="0.035"/>
-      </geometry>
-      <material name="black"/>
-    </visual>
-  </link>
-  <joint name="left_front_wheel_joint" type="continuous">
-    <axis rpy="0 0 0" xyz="0 1 0"/>
-    <parent link="left_base"/>
-    <child link="left_front_wheel"/>
-    <origin rpy="0 0 0" xyz="0.133333333333 0 -0.085"/>
-  </joint>
-  <link name="left_back_wheel">
-    <visual>
-      <origin rpy="1.57075 0 0" xyz="0 0 0"/>
-      <geometry>
-        <cylinder length="0.1" radius="0.035"/>
-      </geometry>
-      <material name="black"/>
-    </visual>
-  </link>
-  <joint name="left_back_wheel_joint" type="continuous">
-    <axis rpy="0 0 0" xyz="0 1 0"/>
-    <parent link="left_base"/>
-    <child link="left_back_wheel"/>
-    <origin rpy="0 0 0" xyz="-0.133333333333 0 -0.085"/>
-  </joint>
-  <joint name="gripper_extension" type="prismatic">
-    <parent link="base_link"/>
-    <child link="gripper_pole"/>
-    <limit effort="1000.0" lower="-0.38" upper="0" velocity="0.5"/>
-    <origin rpy="0 0 0" xyz="0.19 0 0.2"/>
-  </joint>
-  <link name="gripper_pole">
+  <link name="${name}_right_gripper">
     <visual>
       <geometry>
-        <cylinder length="0.2" radius="0.01"/>
+        <box size="${gripper_length} ${gripper_width} ${gripper_height}" />
       </geometry>
-      <origin rpy="0 1.57075 0 " xyz="0.1 0 0"/>
+      <origin xyz="${gripper_length/2} 0 ${gripper_height/2}" />
+      <material name="blue" />
     </visual>
+    <collision>
+      <geometry>
+        <box size="${gripper_length} ${gripper_width} ${gripper_height}" />
+      </geometry>
+      <origin xyz="${gripper_length/2} 0 ${gripper_height/2}" />
+    </collision>
   </link>
-  <joint name="left_gripper_joint" type="revolute">
-    <axis xyz="0 0 1"/>
-    <limit effort="1000.0" lower="0.0" upper="0.548" velocity="0.5"/>
-    <origin rpy="0 0 0" xyz="0.2 0.01 0"/>
-    <parent link="gripper_pole"/>
-    <child link="left_gripper"/>
+  <joint name="${name}_base_joint" type="fixed">
+    <parent link="base_link" />
+    <child link="${name}_base" />
+    <origin xyz="0.5 0 0" rpy="0 ${pi/2} 0" />
   </joint>
-  <link name="left_gripper">
-    <visual>
-      <origin rpy="0.0 0 0" xyz="0 0 0"/>
-      <geometry>
-        <mesh filename="package://urdf_tutorial/meshes/l_finger.dae"/>
-      </geometry>
-    </visual>
-  </link>
-  <joint name="left_tip_joint" type="fixed">
-    <parent link="left_gripper"/>
-    <child link="left_tip"/>
+  <joint name="${name}_shoulder_joint" type="revolute">
+    <parent link="${name}_base" />
+    <child link="${name}_shoulder" />
+    <axis rpy="0 0 0" xyz="0 1 0" />
+    <origin xyz="0 0 ${base_length}" />
+    <limit effort="1000" lower="${-shoulder_limit}" upper="${shoulder_limit}" velocity="1"/>
   </joint>
-  <link name="left_tip">
-    <visual>
-      <origin rpy="0.0 0 0" xyz="0.09137 0.00495 0"/>
-      <geometry>
-        <mesh filename="package://urdf_tutorial/meshes/l_finger_tip.dae"/>
-      </geometry>
-    </visual>
-  </link>
-  <joint name="right_gripper_joint" type="revolute">
-    <axis xyz="0 0 -1"/>
-    <limit effort="1000.0" lower="0.0" upper="0.548" velocity="0.5"/>
-    <origin rpy="0 0 0" xyz="0.2 -0.01 0"/>
-    <parent link="gripper_pole"/>
-    <child link="right_gripper"/>
+  <joint name="${name}_wrist_joint" type="revolute">
+    <parent link="${name}_shoulder" />
+    <child link="${name}_wrist" />
+    <axis rpy="0 0 0" xyz="0 0 1" />
+    <origin xyz="0 0 ${shoulder_length}" />
+    <limit effort="1000" lower="${-wrist_limit}" upper="${wrist_limit}" velocity="1"/>
   </joint>
-  <link name="right_gripper">
-    <visual>
-      <origin rpy="-3.1415 0 0" xyz="0 0 0"/>
-      <geometry>
-        <mesh filename="package://urdf_tutorial/meshes/l_finger.dae"/>
-      </geometry>
-    </visual>
-  </link>
-  <joint name="right_tip_joint" type="fixed">
-    <parent link="right_gripper"/>
-    <child link="right_tip"/>
+  <joint name="${name}_gripper_joint" type="fixed">
+    <parent link="${name}_wrist" />
+    <child link="${name}_gripper" />
+    <origin xyz="0 0 ${gripper_height}" />
   </joint>
-  <link name="right_tip">
-    <visual>
-      <origin rpy="-3.1415 0 0" xyz="0.09137 0.00495 0"/>
-      <geometry>
-        <mesh filename="package://urdf_tutorial/meshes/l_finger_tip.dae"/>
-      </geometry>
-    </visual>
-  </link>
-  <link name="head">
-    <visual>
-      <geometry>
-        <sphere radius="0.2"/>
-      </geometry>
-      <material name="white"/>
-    </visual>
-  </link>
-  <joint name="head_swivel" type="continuous">
-    <parent link="base_link"/>
-    <child link="head"/>
-    <axis xyz="0 0 1"/>
-    <origin xyz="0 0 0.3"/>
+  <joint name="${name}_left_gripper_joint" type="prismatic">
+    <parent link="${name}_wrist" />
+    <child link="${name}_left_gripper" />
+    <axis rpy="0 0 0" xyz="-1 0 0" />
+    <limit effort="1000" lower="0" upper="${gripper_limit}" velocity="1"/>
   </joint>
-  <link name="box">
-    <visual>
-      <geometry>
-        <box size="0.08 0.08 0.08"/>
-      </geometry>
-      <material name="blue"/>
-    </visual>
-  </link>
-  <joint name="tobox" type="fixed">
-    <parent link="head"/>
-    <child link="box"/>
-    <origin xyz="0.1814 0 0.1414"/>
+  <joint name="${name}_right_gripper_joint" type="prismatic">
+    <parent link="${name}_wrist" />
+    <child link="${name}_right_gripper" />
+    <axis rpy="0 0 0" xyz="1 0 0" />
+    <limit effort="1000" lower="0" upper="${gripper_limit}" velocity="1"/>
   </joint>
 </robot>

Commit message: Updates auv_manipulator urdf file

File: src/auv_manipulator/urdf/manipulator.urdf.xacro (robot description, xacro)
@@ -14,5 +14,11 @@
   <xacro:property name="shoulder_limit" value="${(pi/180)*100}" />
   <xacro:property name="wrist_limit" value="${(pi/180)*360}" />
-  <xacro:property name="gripper_limit" value="0.04" />
+  <xacro:property name="gripper_limit" value="${(pi/180)*20}" />
+  <xacro:property name="shoulder_velocity_limit" value="5.0" />
+  <xacro:property name="wrist_velocity_limit" value="5.0" />
+  <xacro:property name="gripper_velocity_limit" value="0.1" />
+  <xacro:property name="shoulder_effort_limit" value="5.0" />
+  <xacro:property name="wrist_effort_limit" value="5.0" />
+  <xacro:property name="gripper_effort_limit" value="0.1" />
   <material name="blue">
     <color rgba="0 0 1 1" />
@@ -132,5 +138,5 @@
     <axis rpy="0 0 0" xyz="0 1 0" />
     <origin xyz="0 0 ${base_length}" />
-    <limit effort="1000" lower="${-shoulder_limit}" upper="${shoulder_limit}" velocity="1"/>
+    <limit effort="${shoulder_effort_limit}" lower="${-shoulder_limit}" upper="${shoulder_limit}" velocity="${shoulder_velocity_limit}"/>
   </joint>
   <joint name="${name}_wrist_joint" type="revolute">
@@ -139,5 +145,5 @@
     <axis rpy="0 0 0" xyz="0 0 1" />
     <origin xyz="0 0 ${shoulder_length}" />
-    <limit effort="1000" lower="${-wrist_limit}" upper="${wrist_limit}" velocity="1"/>
+    <limit effort="${wrist_effort_limit}" lower="${-wrist_limit}" upper="${wrist_limit}" velocity="${wrist_velocity_limit}"/>
   </joint>
   <joint name="${name}_gripper_joint" type="fixed">
@@ -146,15 +152,16 @@
     <origin xyz="0 0 ${gripper_height}" />
   </joint>
-  <joint name="${name}_left_gripper_joint" type="prismatic">
+  <joint name="${name}_left_finger_joint" type="revolute">
     <parent link="${name}_wrist" />
     <child link="${name}_left_gripper" />
-    <axis rpy="0 0 0" xyz="-1 0 0" />
-    <limit effort="1000" lower="0" upper="${gripper_limit}" velocity="1"/>
+    <axis rpy="0 0 0" xyz="0 -1 0" />
+    <limit effort="${gripper_effort_limit}" lower="0" upper="${gripper_limit}" velocity="${gripper_velocity_limit}"/>
   </joint>
-  <joint name="${name}_right_gripper_joint" type="prismatic">
+  <joint name="${name}_right_finger_joint" type="revolute">
     <parent link="${name}_wrist" />
     <child link="${name}_right_gripper" />
-    <axis rpy="0 0 0" xyz="1 0 0" />
-    <limit effort="1000" lower="0" upper="${gripper_limit}" velocity="1"/>
+    <axis rpy="0 0 0" xyz="0 1 0" />
+    <limit effort="${gripper_effort_limit}" lower="0" upper="${gripper_limit}" velocity="${gripper_velocity_limit}"/>
+    <mimic joint="twig_left_finger_joint" />
   </joint>
 </robot>

Commit message: Updates twig gripper velocity limits

File: src/auv_manipulator/urdf/manipulator.urdf.xacro (robot description, xacro)
@@ -17,5 +17,5 @@
   <xacro:property name="shoulder_velocity_limit" value="5.0" />
   <xacro:property name="wrist_velocity_limit" value="5.0" />
-  <xacro:property name="gripper_velocity_limit" value="0.1" />
+  <xacro:property name="gripper_velocity_limit" value="1.0" />
   <xacro:property name="shoulder_effort_limit" value="5.0" />
   <xacro:property name="wrist_effort_limit" value="5.0" />
