Commit message: Reverses direction or twig shoulder and wrist axis

File: src/twig_description/urdf/twig.urdf.xacro (robot description, xacro)
@@ -136,5 +136,5 @@
     <parent link="${name}_base" />
     <child link="${name}_shoulder" />
-    <axis rpy="0 0 0" xyz="0 1 0" />
+    <axis rpy="0 0 0" xyz="0 -1 0" />
     <origin xyz="0 0 ${base_length}" />
     <limit effort="${shoulder_effort_limit}" lower="${-shoulder_limit}" upper="${shoulder_limit}" velocity="${shoulder_velocity_limit}"/>
@@ -143,5 +143,5 @@
     <parent link="${name}_shoulder" />
     <child link="${name}_wrist" />
-    <axis rpy="0 0 0" xyz="0 0 1" />
+    <axis rpy="0 0 0" xyz="0 0 -1" />
     <origin xyz="0 0 ${shoulder_length}" />
     <limit effort="${wrist_effort_limit}" lower="${-wrist_limit}" upper="${wrist_limit}" velocity="${wrist_velocity_limit}"/>
